File: design_files/NTB.kicad_sch (KiCad schematic)
At the start: 124 parts, among them U1 DEV-16771, U2 ADS131M02IPWR, U3 ADP7118AUJZ-3.3-R7, U4 ADP7118AUJZ-3.3-R7, U5 DAC8831ID, U6 DAC8831ID, Y1 SG-8018CE 2.048000MHz TJHPA

Commit message: Add files via upload
Connections:
- net GND_Sense: now also B6252H5-NPP3G-1. (GND), B6252H5-NPP3G-2. (GND)
- net GND_Stim: now also B6252H5-NPP3G-3. (GND), B6252H5-NPP3G-4. (GND)
- no-connect marks 21 -> 13
