File: design_files/NTB_schematic.kicad_sch (KiCad schematic)
At the start: 186 parts, among them IC1 ADP7118AUJZ-3.3-R7, IC10 OPA192IDGKT, IC11 OPA2192IDR_BKN, IC15 ADP7118AUJZ-5.0-R7, IC16 ADP7118AUJZ-5.0-R7, IC17 ADP7118AUJZ-R7, IC18 ADP7118AUJZ-5.0-R7, IC19 SI8660BC-B-IS1, IC2 ADP7118AUJZ-5.0-R7, IC20 SI8660BC-B-IS1R, IC21 TXU0101DCKR, IC22 TXU0101DCKR, IC23 OPA2192IDR_BKN, IC24 ADC122S051CIMM_NOPB, IC25 OPA2192IDR_BKN, IC26 OPA2192IDR_BKN, IC27 OPA2192IDR_BKN, IC28 OPA192IDGKT, IC3 ADP7118AUJZ-R7, IC4 ADP7118AUJZ-3.3-R7, IC5 SI8660BC-B-IS1, IC6 SI8660BC-B-IS1R, IC7 ADS131M02IPWR, IC8 TMUX6112PWR, IC9 OPA2192IDR_BKN, J4 CH1, J5 CH2, U1 DEV-16771

Commit message: updated designators to match pictures from Mo
Parts:
- C19: renamed from C18; value ~ -> (none); now left out of the parts list
- C23: renamed from C86; now left out of the parts list
- C25: renamed from C87; now left out of the parts list
- C33: renamed from C75; now left out of the parts list
- C35: renamed from C19; value ~ -> (none); now left out of the parts list
- C41: renamed from C76; now left out of the parts list
- C58: renamed from C37; now left out of the parts list
- C72: renamed from C71; now left out of the parts list
- C77: renamed from C47; now left out of the parts list
- C78: renamed from C44; now left out of the parts list
- C79: renamed from C52; value ~ -> (none); now left out of the parts list
- C80: renamed from C51; value ~ -> (none); now left out of the parts list
- C82: renamed from C36; now left out of the parts list
- IC1: renamed from IC8; now left out of the parts list
- IC13: renamed from IC24; now left out of the parts list
- IC8: renamed from U1; value DEV-16771 -> TEENSY_4.1
- J2: renamed from J1; value ~ -> (none)
- J3: renamed from J2; value ~ -> (none)
- J4: renamed from J3; value ~ -> (none)
- LED1, LEDS1, S1: now left out of the parts list
- R21: renamed from R4; now left out of the parts list
- R27: renamed from R3; now left out of the parts list
- R28: renamed from R23; now left out of the parts list
- R29: renamed from R5; now left out of the parts list
- R30: renamed from R22; now left out of the parts list
- R58: renamed from R26; now left out of the parts list
- S3: renamed from S2; now left out of the parts list
- SJ2: renamed from JP3; value ~ -> (none)
- SJ3: renamed from JP1; value ~ -> (none)
- TTL_IN: value ~ -> (none); now left out of the parts list
- Y1: renamed from Y2; value ~ -> SG-8018CE_2.0000M-TJHPA3
- renumbered C8 to C1, C39 to C10, C78 to C11, C79 to C12, C80 to C13, C82 to C14, C81 to C15, C83 to C16, C84 to C17, C85 to C18, C61 to C2, C4 to C20, C57 to C21, C14 to C22, C60 to C24, C22 to C26, C21 to C27, C20 to C28, C27 to C29, C63 to C3, C26 to C30, C16 to C31, C64 to C32, C38 to C34, C55 to C36, C72 to C37, C40 to C38, C73 to C39, C70 to C4, C74 to C40, C11 to C42, C13 to C43, C7 to C44, C29 to C45, C32 to C46, C30 to C47, C31 to C48, C34 to C49, C15 to C5, C35 to C50, C33 to C51, C6 to C52, C59 to C53, C69 to C54, C62 to C55, C68 to C56, C66 to C57, C24 to C59, C17 to C6, C48 to C60, C41 to C61, C2 to C62, C3 to C63, C28 to C64, C49 to C65, C1 to C66, C54 to C67, C10 to C68, C9 to C69, C5 to C7, C45 to C70, C53 to C71, C42 to C73, C46 to C74, C50 to C75, C43 to C76, C58 to C8, C25 to C81, C67 to C83, C65 to C84, C12 to C87, C23 to C88, C77 to C9, DAC2 to DAC3, IC16 to IC10, IC3 to IC11, IC7 to IC12, IC11 to IC14, IC9 to IC15, IC23 to IC17, IC15 to IC18, IC1 to IC19, IC26 to IC2, IC4 to IC20, IC18 to IC21, IC6 to IC22, IC28 to IC23, IC2 to IC24, IC17 to IC25, IC10 to IC28, IC27 to IC3, IC19 to IC4, IC20 to IC6, IC5 to IC7, IC25 to IC9, J4 to J5, J5 to J6, L3 to L1, L4 to L2, PS2 to PS3, R40 to R1, R13 to R10, R12 to R11, R6 to R12, R59 to R13, R58 to R14, R60 to R15, R61 to R16, R57 to R17, R62 to R18, R63 to R19, R41 to R2, R64 to R20, R46 to R22, R42 to R23, R43 to R24, R45 to R25, R2 to R26, R51 to R3, R48 to R31, R47 to R32, R50 to R33, R8 to R34, R9 to R35, R44 to R36, R49 to R37, R1 to R38, R7 to R39, R52 to R4, R29 to R43, R30 to R44, R27 to R45, R28 to R46, R18 to R47, R14 to R48, R25 to R49, R54 to R5, R24 to R50, R17 to R51, R19 to R52, R21 to R53, R20 to R54, R15 to R55, R16 to R57, R53 to R6, R55 to R7, R11 to R8, R10 to R9
Connections:
- net GND_Arduino is gone; now on net GND: C2.2
- net GND: no longer C10.1, C11.1, C12.1, C13.1, C14.1, C15.1, C16.1, C17.1, C20.1, C21.2, C23.1, C24.2, C25.1, C28.2, C29.1, C3.2, C30.2, C32.2, C33.2, C34.1, C36.1, C37.1, C38.1, C39.1, C4.1, C40.1, C41.2, C42.1, C43.2, C44.2, C45.2, C47.2, C48.1, C5.1, C50.2, C51.1, C52.1, C53.2, C54.2, C55.1, C58.2, C59.1, C6.2, C60.1, C61.1, C62.2, C63.2, C64.2, C65.1, C66.2, C67.1, C69.2, C7.1, C70.1, C71.1, C73.1, C74.1, C75.1, C77.1, C78.1, C8.2, C81.2, C82.2, C87.1, C88.2, C9.1, DAC3. (SCLK), IC1.5 (GND), IC10.2 (GND), IC11.1 (GND), IC13.3 (GND), IC17.5 (+IN_B), IC18.2 (GND), IC19.2 (GND), IC20.2 (GND), IC21.2 (GND), IC22.9 (GND2), IC24.2 (GND), IC25.1 (GND), IC4.9 (GND2), IC6.9 (GND2), IC7.9 (GND2), IC9.5 (+IN_B), J5.2, J6.2, PS3.7 (0V), R13.2, R2.1, R20.1, R21.1, R24.1, R27.1, R28.1, R29.2, R30.2, R35.1, R39.1, R46.2, R48.1, R49.2, R56.1, R57.1, R58.1, R6.2, S1.3 (GND), S3.3 (GND), Y1.2 (GND)
- net GND_sense: now reaches C27.1, R12.1
- net GND_sense: now also C28.2, C29.1, C30.2, C42.1, C43.2, C44.2, C45.2, C47.2, C48.1, C50.2, C51.1, C58.2, C59.1, C62.2, C63.2, C64.2, C66.2, C69.2, C81.2, C82.2, C87.1, C88.2, IC1.5 (GND), IC11.1 (GND), IC12. (CS), IC19.2 (GND), IC20.2 (GND), IC22.9 (GND2), IC24.2 (GND), IC7.9 (GND2), PS3.7 (0V), R35.1, R39.1, Y1.2 (GND)
- new net GND_sig: C10.1, C11.1, C12.1, C13.1, C14.1, C15.1, C16.1, C17.1, C20.1, C21.2, C23.1, C24.2, C25.1, C3.2, C32.2, C33.2, C34.1, C36.1, C37.1, C38.1, C39.1, C4.1, C40.1, C41.2, C5.1, C52.1, C53.2, C54.2, C55.1, C6.2, C60.1, C61.1, C65.1, C67.1, C7.1, C70.1, C71.1, C73.1, C74.1, C75.1, C77.1, C78.1, C8.2, C9.1, DAC3. (SCLK), IC10.2 (GND), IC13.3 (GND), IC17.5 (+IN_B), IC18.2 (GND), IC21.2 (GND), IC25.1 (GND), IC4.9 (GND2), IC6.9 (GND2), IC9.5 (+IN_B), J5.2, J6.2, R13.2, R2.1, R20.1, R21.1, R24.1, R27.1, R28.1, R29.2, R30.2, R46.2, R48.1, R49.2, R56.1, R57.1, R58.1, R6.2, S1.3 (GND), S3.3 (GND)
Other:
- note removed: "VDDA+ = 5V(1+R1/R7) VDDA+ = 5V(1+6.2/10) VDDA+ = 5V(1.6) = +8.1V"
- note removed: "VDDA+ = 5V(1+R42/R43) VDDA+ = 5V(1+18/10) VDDA+ = 5V(2.8) = +14V"
- note removed: "VDDA- = -1.22V(1+R40/R41) VDDA- = -1.22V(1+10.5/1) VDDA- = -1.22V(11.5) = -14.03V"
- note removed: "VDDA- = -1.22V(1+R8/R9) VDDA- = -1.22V(1+5.6/1) VDDA- = -1.22V(6.6) = -8V"
- moved on the sheet: C46, C47, C48, C49, C50, C51, R10, R11, R8, R9
